File: PCB_Rev2/PH-AC.kicad_sch (KiCad schematic)
At the start: 44 parts, among them J1 USB_C_Receptacle_USB2.0_14P, J2 Conn_01x03, Q1 DMG1012T, SW1 SW_Push, U1 RP2040, U2 RT6150B-33GQW, U3 W25Q16JVSS, Y1 Crystal_GND24

Commit message: Mouting Hole Adding
Parts:
- added H1, H2, H3, H4, H5, H6, H7, H8: MountingHole, MountingHole:MountingHole_3.2mm_M3_ISO7380_Pad, symbol Mechanical:MountingHole

Commit message: Component Package Modification
Parts:
- D1: footprint Diode_SMD:D_0402_1005Metric -> Diode_SMD:D_SOD-123F
Changed lines of the file:
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@@
 			)
 		)
-		(property "Footprint" "Diode_SMD:D_0402_1005Metric"
+		(property "Footprint" "Diode_SMD:D_SOD-123F"
 			(at 104.14 200.66 0)
 			(effects
