File: PCB_Rev2.1/PH-AC.kicad_sch (KiCad schematic)
At the start: 52 parts, among them J1 USB_C_Receptacle_USB2.0_14P, J2 Conn_01x03, Q1 DMG1012T, SW1 SW_Push, U1 RP2040, U2 RT6150B-33GQW, U3 W25Q16JVSS, Y1 Crystal_GND24

Commit message: Minor Update
Fixed wiring mistake of D+ and D-.
Decreased the thickness of upper panel to 1.4mm
Connections:
- net USB_DM: now also R4.1; no longer R3.1
- net USB_DP: now also R3.1; no longer R4.1
Changed lines of the file:
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@@
 		)
 	)
-	(label "USB_DM"
+	(label "USB_DP"
 		(at 259.08 135.89 0)
 		(fields_autoplaced yes)
@@
 		)
 	)
-	(label "USB_DP"
+	(label "USB_DM"
 		(at 259.08 146.05 0)
 		(fields_autoplaced yes)

Commit message: Case Improvement
Parts:
- D1: value D_Schottky -> MBR120VLSFT1G
Changed lines of the file:
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@@
 			)
 		)
-		(property "Value" "D_Schottky"
+		(property "Value" "MBR120VLSFT1G"
 			(at 104.4575 196.85 0)
 			(effects

Commit message: Design Modification
Connections:
- net ENC1A: now also U1.9 (GPIO7); no longer U1.8 (GPIO6)
- net ENC1B: now also U1.11 (GPIO8); no longer U1.9 (GPIO7)
- net ENC2A: now also U1.13 (GPIO10); no longer U1.11 (GPIO8)
- net COL0 renamed BT6
- net COL1 renamed BT5
- net COL2 renamed BT4
- net COL3 renamed BT3
- net ROW0 renamed BT2
- net ROW1 renamed BT1
- new net BT0: U1.8 (GPIO6)
- no-connect marks 17 -> 16
Changed lines of the file:
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@@
-	)
-	(no_connect
-		(at 327.66 157.48)
 	)
 	(no_connect
@@
 		)
 	)
-	(global_label "ENC2A"
-		(shape input)
-		(at 327.66 152.4 0)
-		(fields_autoplaced yes)
-		(effects
-			(font
-				(size 1.27 1.27)
-			)
-			(justify left)
-		)
-		(property "Intersheetrefs" "${INTERSHEET_REFS}"
-			(at 336.6928 152.4 0)
-			(effects
-				(font
-					(size 1.27 1.27)
-				)
-				(justify left)
-				(hide yes)
-			)
-		)
-	)
-	(global_label "COL2"
-		(shape input)
-		(at 327.66 137.16 0)
-		(fields_autoplaced yes)
-		(effects
-			(font
-				(size 1.27 1.27)
-			)
-			(justify left)
-		)
-		(property "Intersheetrefs" "${INTERSHEET_REFS}"
-			(at 335.4833 137.16 0)
-			(effects
-				(font
-					(size 1.27 1.27)
-				)
-				(justify left)
-				(hide yes)
-			)
-		)
-	)
-	(global_label "ROW0"
-		(shape input)
-		(at 327.66 142.24 0)
-		(fields_autoplaced yes)
-		(effects
-			(font
-				(size 1.27 1.27)
-			)
-			(justify left)
-		)
-		(property "Intersheetrefs" "${INTERSHEET_REFS}"
-			(at 335.9066 142.24 0)
-			(effects
-				(font
-					(size 1.27 1.27)
-				)
-				(justify left)
-				(hide yes)
-			)
-		)
-	)
-	(global_label "ENC1B"
-		(shape input)
-		(at 327.66 149.86 0)
-		(fields_autoplaced yes)
-		(effects
-			(font
-				(size 1.27 1.27)
-			)
-			(justify left)
-		)
-		(property "Intersheetrefs" "${INTERSHEET_REFS}"
-			(at 336.8742 149.86 0)
-			(effects
-				(font
-					(size 1.27 1.27)
-				)
-				(justify left)
-				(hide yes)
-			)
-		)
-	)
-	(global_label "COL1"
-		(shape input)
-		(at 327.66 134.62 0)
-		(fields_autoplaced yes)
-		(effects
-			(font
-				(size 1.27 1.27)
-			)
-			(justify left)
-		)
-		(property "Intersheetrefs" "${INTERSHEET_REFS}"
-			(at 335.4833 134.62 0)
-			(effects
-				(font
-					(size 1.27 1.27)
-				)
-				(justify left)
-				(hide yes)
-			)
-		)
-	)
-	(global_label "COL0"
-		(shape input)
-		(at 327.66 132.08 0)
-		(fields_autoplaced yes)
-		(effects
-			(font
-				(size 1.27 1.27)
-			)
-			(justify left)
-		)
-		(property "Intersheetrefs" "${INTERSHEET_REFS}"
-			(at 335.4833 132.08 0)
-			(effects
-				(font
-					(size 1.27 1.27)
-				)
-				(justify left)
-				(hide yes)
-			)
-		)
-	)
-	(global_label "ROW1"
+	(global_label "BT1"
 		(shape input)
 		(at 327.66 144.78 0)
@@
 		)
 		(property "Intersheetrefs" "${INTERSHEET_REFS}"
-			(at 335.9066 144.78 0)
+			(at 334.0923 144.78 0)
 			(effects
 				(font
@@
 		)
 	)
-	(global_label "COL3"
+	(global_label "BT2"
 		(shape input)
-		(at 327.66 139.7 0)
+		(at 327.66 142.24 0)
 		(fields_autoplaced yes)
 		(effects
@@
 		)
 		(property "Intersheetrefs" "${INTERSHEET_REFS}"
-			(at 335.4833 139.7 0)
+			(at 334.0923 142.24 0)
 			(effects
 				(font
@@
 		)
 	)
+	(global_label "BT6"
+		(shape input)
+		(at 327.66 132.08 0)
+		(fields_autoplaced yes)
+		(effects
+			(font
+				(size 1.27 1.27)
+			)
+			(justify left)
+		)
+		(property "Intersheetrefs" "${INTERSHEET_REFS}"
+			(at 334.0923 132.08 0)
+			(effects
+				(font
+					(size 1.27 1.27)
+				)
+				(justify left)
+				(hide yes)
+			)
+		)
+	)
+	(global_label "BT4"
+		(shape input)
+		(at 327.66 137.16 0)
+		(fields_autoplaced yes)
+		(effects
+			(font
+				(size 1.27 1.27)
+			)
+			(justify left)
+		)
+		(property "Intersheetrefs" "${INTERSHEET_REFS}"
+			(at 334.0923 137.16 0)
+			(effects
+				(font
+					(size 1.27 1.27)
+				)
+				(justify left)
+				(hide yes)
+			)
+		)
+	)
+	(global_label "ENC1B"
+		(shape input)
+		(at 327.66 152.4 0)
+		(fields_autoplaced yes)
+		(effects
+			(font
+				(size 1.27 1.27)
+			)
+			(justify left)
+		)
+		(property "Intersheetrefs" "${INTERSHEET_REFS}"
+			(at 336.8742 152.4 0)
+			(effects
+				(font
+					(size 1.27 1.27)
+				)
+				(justify left)
+				(hide yes)
+			)
+		)
+	)
+	(global_label "BT3"
+		(shape input)
+		(at 327.66 139.7 0)
+		(fields_autoplaced yes)
+		(effects
+			(font
+				(size 1.27 1.27)
+			)
+			(justify left)
+		)
+		(property "Intersheetrefs" "${INTERSHEET_REFS}"
+			(at 334.0923 139.7 0)
+			(effects
+				(font
+					(size 1.27 1.27)
+				)
+				(justify left)
+				(hide yes)
+			)
+		)
+	)
+	(global_label "BT5"
+		(shape input)
+		(at 327.66 134.62 0)
+		(fields_autoplaced yes)
+		(effects
+			(font
+				(size 1.27 1.27)
+			)
+			(justify left)
+		)
+		(property "Intersheetrefs" "${INTERSHEET_REFS}"
+			(at 334.0923 134.62 0)
+			(effects
+				(font
+					(size 1.27 1.27)
+				)
+				(justify left)
+				(hide yes)
+			)
+		)
+	)
+	(global_label "ENC2A"
+		(shape input)
+		(at 327.66 157.48 0)
+		(fields_autoplaced yes)
+		(effects
+			(font
+				(size 1.27 1.27)
+			)
+			(justify left)
+		)
+		(property "Intersheetrefs" "${INTERSHEET_REFS}"
+			(at 336.6928 157.48 0)
+			(effects
+				(font
+					(size 1.27 1.27)
+				)
+				(justify left)
+				(hide yes)
+			)
+		)
+	)
+	(global_label "BT0"
+		(shape input)
+		(at 327.66 147.32 0)
+		(fields_autoplaced yes)
+		(effects
+			(font
+				(size 1.27 1.27)
+			)
+			(justify left)
+		)
+		(property "Intersheetrefs" "${INTERSHEET_REFS}"
+			(at 334.0923 147.32 0)
+			(effects
+				(font
+					(size 1.27 1.27)
+				)
+				(justify left)
+				(hide yes)
+			)
+		)
+	)
 	(global_label "ENC1A"
 		(shape input)
-		(at 327.66 147.32 0)
+		(at 327.66 149.86 0)
 		(fields_autoplaced yes)
 		(effects
@@
 		)
 		(property "Intersheetrefs" "${INTERSHEET_REFS}"
-			(at 336.6928 147.32 0)
+			(at 336.6928 149.86 0)
 			(effects
 				(font
