File: PCB_Rev2.1/matrix.kicad_sch (KiCad schematic)
At the start: 16 parts, among them SW10 SW_Push, SW2 RotaryEncoder_Switch_MP, SW3 RotaryEncoder_Switch_MP, SW4 SW_Push, SW5 SW_Push, SW6 SW_Push, SW7 SW_Push, SW8 SW_Push, SW9 SW_Push

Commit message: Detail Improvement
Changed the package size of diodes from 0402 to 0805.
Parts:
- D3, D4, D5, D6, D7, D8, D9: footprint Diode_SMD:D_0402_1005Metric -> Diode_SMD:D_0805_2012Metric
- SW10, SW8: footprint PCM_Switch_Keyboard_Hotswap_Kailh:SW_Hotswap_Kailh_MX_2.75u -> PCM_Switch_Keyboard_Hotswap_Kailh:SW_Hotswap_Kailh_MX_2.25u
Changed lines of the file:
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@@
 			)
 		)
-		(property "Footprint" "Diode_SMD:D_0402_1005Metric"
+		(property "Footprint" "Diode_SMD:D_0805_2012Metric"
 			(at 44.45 107.95 0)
 			(effects
@@
 			)
 		)
-		(property "Footprint" "Diode_SMD:D_0402_1005Metric"
+		(property "Footprint" "Diode_SMD:D_0805_2012Metric"
 			(at 59.69 88.9 0)
 			(effects
@@
 			)
 		)
-		(property "Footprint" "PCM_Switch_Keyboard_Hotswap_Kailh:SW_Hotswap_Kailh_MX_2.75u"
+		(property "Footprint" "PCM_Switch_Keyboard_Hotswap_Kailh:SW_Hotswap_Kailh_MX_2.25u"
 			(at 80.01 99.06 0)
 			(effects
@@
 			)
 		)
-		(property "Footprint" "PCM_Switch_Keyboard_Hotswap_Kailh:SW_Hotswap_Kailh_MX_2.75u"
+		(property "Footprint" "PCM_Switch_Keyboard_Hotswap_Kailh:SW_Hotswap_Kailh_MX_2.25u"
 			(at 49.53 99.06 0)
 			(effects
@@
 			)
 		)
-		(property "Footprint" "Diode_SMD:D_0402_1005Metric"
+		(property "Footprint" "Diode_SMD:D_0805_2012Metric"
 			(at 74.93 88.9 0)
 			(effects
@@
 			)
 		)
-		(property "Footprint" "Diode_SMD:D_0402_1005Metric"
+		(property "Footprint" "Diode_SMD:D_0805_2012Metric"
 			(at 90.17 88.9 0)
 			(effects
@@
 			)
 		)
-		(property "Footprint" "Diode_SMD:D_0402_1005Metric"
+		(property "Footprint" "Diode_SMD:D_0805_2012Metric"
 			(at 74.93 107.95 0)
 			(effects
@@
 			)
 		)
-		(property "Footprint" "Diode_SMD:D_0402_1005Metric"
+		(property "Footprint" "Diode_SMD:D_0805_2012Metric"
 			(at 59.69 107.95 0)
 			(effects
@@
 			)
 		)
-		(property "Footprint" "Diode_SMD:D_0402_1005Metric"
+		(property "Footprint" "Diode_SMD:D_0805_2012Metric"
 			(at 44.45 88.9 0)
 			(effects

Commit message: Design Modification
Parts:
- removed D3, D4, D5, D6, D7, D8, D9: D, Diode_SMD:D_0805_2012Metric, symbol Device:D
Connections:
- net COL0 is gone; now on net GND: SW4.2, SW8.2
- net COL1 is gone; now on net GND: SW5.2, SW9.2
- net COL2 is gone; now on net GND: SW10.2, SW6.2
- net COL3 is gone; now on net GND: SW7.2
- net ENC1A: now also SW3.A; no longer SW2.A
- net ENC1B: now also SW3.B; no longer SW2.B
- net ENC2A: now also SW2.A; no longer SW3.A
- net ENC2B: now also SW2.B; no longer SW3.B
- net BT0: now reaches SW4.1
- net BT1: now reaches SW5.1
- net BT4: now reaches SW8.1
- net BT6: now reaches SW10.1
- net BT2: now reaches SW6.1
- net BT3: now reaches SW7.1
- net BT5: now reaches SW9.1
Other:
- moved on the sheet: SW10, SW5, SW6, SW7, SW9
